Commit message: launch two robots

File: turtlebot_follows_turtlebot_description/urdf/turtlebot3_waffle_pi_aruco.urdf.xacro (robot description, xacro)
@@ -13,7 +13,7 @@
       <origin xyz="-0.064 0 0.0" rpy="0 0 0"/>
       <geometry>
-        <mesh filename="package://turtlebot_follows_turtlebot_description/meshes/3x3_floor_marker.dae" scale="1 1 1"/>
-      </geometry>
-      <!-- <material name="light_black"/> -->
+        <mesh filename="package://turtlebot3_description/meshes/bases/waffle_pi_base.stl" scale="0.001 0.001 0.001"/>
+      </geometry>
+      <material name="light_black"/>
     </visual>
     <collision>
@@ -31,4 +31,19 @@
     </inertial>
   </link>
+  <!-- ArUco -->
+  <joint name="aruco_joint" type="fixed">
+      <parent link="base_link"/>
+      <child link="aruco_link" />
+      <origin xyz="-0.2 0 0.08" rpy="0 -1.57 0"/>
+  </joint>
+  <link name="aruco_link">
+      <visual>
+          <origin xyz="0 0 0" rpy="0 0 0"/>
+          <geometry>
+              <mesh filename="package://turtlebot_follows_turtlebot_description/meshes/aruco_board.dae" scale="0.15 0.15 0.15"/>
+          </geometry>
+          <material name="light_black"/>
+      </visual>
+  </link>
   <joint name="wheel_left_joint" type="continuous">
     <parent link="base_link"/>
